File: Display/Display_v5.sch (EAGLE design)
At the start: 11 parts

Commit message: Resolved switched pins issue
Connections:
- removed net N$1: JP1.2, U$1.0
- removed net N$10: JP1.20, U$1.9
- removed net N$13: JP1.26, U$2.2
- removed net N$14: JP1.28, U$2.3
- removed net N$15: JP1.30, U$2.4
- removed net N$16: JP1.32, U$2.5
- removed net N$17: JP1.34, U$2.6
- removed net N$18: JP1.36, U$2.7
- removed net N$19: JP1.38, U$2.8
- removed net N$20: JP1.40, U$2.9
- removed net N$31: JP1.21, U$4.9
- removed net N$32: JP1.23, U$4.8
- removed net N$33: JP1.25, U$4.7
- removed net N$34: JP1.27, U$4.6
- removed net N$35: JP1.29, U$4.5
- removed net N$36: JP1.31, U$4.4
- removed net N$37: JP1.33, U$4.3
- removed net N$38: JP1.35, U$4.2
- removed net N$39: JP1.37, U$4.1
- removed net N$4: JP1.8, U$1.3
- removed net N$40: JP1.39, U$4.0
- removed net N$7: JP1.14, U$1.6
- removed net N$8: JP1.16, U$1.7
- removed net N$9: JP1.18, U$1.8
- new net N$43: JP1.14, U$1.3
- new net N$44: JP1.16, U$1.2
- new net N$50: JP1.18, U$1.1
- new net N$51: JP1.20, U$1.0
- new net N$52: JP1.38, U$2.1
- new net N$53: JP1.36, U$2.2
- new net N$54: JP1.34, U$2.3
- new net N$56: JP1.24, U$2.8
- new net N$57: JP1.26, U$2.7
- new net N$58: JP1.28, U$2.6
- new net N$59: JP1.30, U$2.5
- new net N$60: JP1.32, U$2.4
- new net N$61: JP1.2, U$1.9
- new net N$64: JP1.8, U$1.6
- new net N$65: JP1.10, U$1.5
- new net N$66: JP1.12, U$1.4
- new net N$77: JP1.37, U$4.8
- new net N$78: JP1.35, U$4.7
- new net N$79: JP1.33, U$4.6
- new net N$80: JP1.31, U$4.5
- new net N$81: JP1.29, U$4.4
- new net N$82: JP1.27, U$4.3
- new net N$83: JP1.25, U$4.2
- new net N$85: JP1.21, U$4.0
- net N$11: now also JP1.40; no longer JP1.22
- net N$12: now also JP1.22, U$2.9; no longer JP1.24, U$2.1
- net N$2: now also JP1.23, U$4.1; no longer JP1.4, U$1.1
- net N$21: now also JP1.19; no longer JP1.1
- net N$22: now also JP1.17; no longer JP1.3
- net N$23: now also JP1.15; no longer JP1.5
- net N$24: now also JP1.13; no longer JP1.7
- net N$25: now also JP1.11; no longer JP1.9
- net N$26: now also JP1.9; no longer JP1.11
- net N$27: now also JP1.7; no longer JP1.13
- net N$28: now also JP1.5; no longer JP1.15
- net N$29: now also JP1.3; no longer JP1.17
- net N$3: now also JP1.39, U$4.9; no longer JP1.6, U$1.2
- net N$30: now also JP1.1; no longer JP1.19
- net N$5: now also JP1.4, U$1.8; no longer JP1.10, U$1.4
- net N$6: now also JP1.6, U$1.7; no longer JP1.12, U$1.5
Other:
- moved on the sheet: R2, R3
